File: YAPoco/YAPoco.kicad_sch (KiCad schematic)
At the start: 18 parts, among them P1 Cart Connector, U1 CGB CPU, U6 PST9135N, X1 Crystal_Small

Commit message: updated some labels
Changed lines of the file:
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@@
 		(dnp no)
 		(property "Reference" "U1"
-			(at 209.55 71.8708 0)
+			(at 222.25 54.7258 0)
 			(effects
 				(font
@@
 		)
 		(property "Value" "CGB CPU"
-			(at 209.55 74.295 0)
+			(at 222.25 57.15 0)
 			(effects
 				(font
