File: KiCad Files/CGB_Serial.kicad_sch (KiCad schematic)
At the start: 10 parts, among them P3 Conn_01x06

Commit message: fixed some BOM stuff
Parts:
- P3: value Conn_01x06 -> Serial Port; now left out of the parts list
- RA3: value 270 -> 270R
Other:
- title: CGB Reverse Engineer -> Yet Another Pocket Color (YAP)
