File: KiCad Files/CGB_Sound.kicad_sch (KiCad schematic)
At the start: 21 parts, among them P5 Conn_01x05, U3 MGB AMP

Commit message: fixed some BOM stuff
Parts:
- P5: value Conn_01x05 -> Headphone Jack; now left out of the parts list
- RA1: value R_Pack02_SIP_Split -> 510R
- RA2: value R_Pack02_SIP_Split -> 15R
- SP1, U3: now left out of the parts list
- VR1: value Conn_01x05 -> 10K Dual Thumbwheel Potentiometer
Other:
- title: CGB Reverse Engineer -> Yet Another Pocket Color (YAP)
