File: KiCad Files/YAPoco.kicad_sch (KiCad schematic)
At the start: 18 parts, among them P1 Cart Connector, U1 CGB CPU, U6 PST9135N, X1 Crystal_Small

Commit message: fixed some BOM stuff
Parts:
- C46: value ~ -> DNP; now not fitted
- P1, U1: now left out of the parts list
- U2: value ~ -> CGB SRAM
- X1: value Crystal_Small -> 8.388608MHZ
Other:
- title: CGB Reverse Engineer -> Yet Another Pocket Color (YAP)
Changed lines of the file:
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@@
 (kicad_sch
-	(version 20231120)
+	(version 20250114)
 	(generator "eeschema")
-	(generator_version "8.0")
+	(generator_version "9.0")
 	(paper "A4")
 	(title_block
-		(title "CGB Reverse Engineer")
+		(title "Yet Another Pocket Color (YAP)")
 		(company "NatalieTheNerd.com")
 	)
+	(text "Not always populated"
+		(exclude_from_sim no)
+		(at 239.395 48.895 0)
+		(effects
+			(font
+				(size 1.27 1.27)
+			)
+			(justify left bottom)
+		)
+	)
+	(text "Low reset type IC"
+		(exclude_from_sim no)
+		(at 41.275 177.165 0)
+		(effects
+			(font
+				(size 1.27 1.27)
+			)
+			(justify left bottom)
+		)
+	)
+	(text "SRAM"
+		(exclude_from_sim no)
+		(at 160.02 141.605 0)
+		(effects
+			(font
+				(size 1.27 1.27)
+			)
+			(justify left bottom)
+		)
+	)
 	(junction
 		(at 48.26 155.575)
@@
 		)
 	)
-	(text "Not always populated"
-		(exclude_from_sim no)
-		(at 239.395 48.895 0)
-		(effects
-			(font
-				(size 1.27 1.27)
-			)
-			(justify left bottom)
-		)
-	)
-	(text "Low reset type IC"
-		(exclude_from_sim no)
-		(at 41.275 177.165 0)
-		(effects
-			(font
-				(size 1.27 1.27)
-			)
-			(justify left bottom)
-		)
-	)
-	(text "SRAM"
-		(exclude_from_sim no)
-		(at 160.02 141.605 0)
-		(effects
-			(font
-				(size 1.27 1.27)
-			)
-			(justify left bottom)
-		)
-	)
 	(label "D6"
 		(at 46.355 116.84 0)
-		(fields_autoplaced yes)
 		(effects
 			(font
@@
 	(label "RD"
 		(at 46.355 55.88 0)
-		(fields_autoplaced yes)
 		(effects
 			(font
@@
 	(label "D3"
 		(at 46.355 109.22 0)
-		(fields_autoplaced yes)
 		(effects
 			(font
@@
 	(label "A12"
 		(at 46.355 91.44 0)
-		(fields_autoplaced yes)
 		(effects
 			(font
@@
 	(label "A10"
 		(at 46.355 86.36 0)
-		(fields_autoplaced yes)
 		(effects
 			(font
@@
 	(label "D5"
 		(at 46.355 114.3 0)
-		(fields_autoplaced yes)
 		(effects
 			(font
@@
 	(label "D1"
 		(at 46.355 104.14 0)
-		(fields_autoplaced yes)
 		(effects
 			(font
@@
 	(label "RESET"
 		(at 46.355 121.92 0)
-		(fields_autoplaced yes)
 		(effects
 			(font
@@
 	(label "A9"
 		(at 46.355 83.82 0)
-		(fields_autoplaced yes)
 		(effects
 			(font
@@
 	(label "D0"
 		(at 46.355 101.6 0)
-		(fields_autoplaced yes)
 		(effects
 			(font
@@
 	(label "A13"
 		(at 46.355 93.98 0)
-		(fields_autoplaced yes)
 		(effects
 			(font
@@
 	(label "CS"
 		(at 46.355 58.42 0)
-		(fields_autoplaced yes)
 		(effects
 			(font
@@
 	(label "A14"
 		(at 46.355 96.52 0)
-		(fields_autoplaced yes)
 		(effects
 			(font
@@
 	(label "A11"
 		(at 46.355 88.9 0)
-		(fields_autoplaced yes)
 		(effects
 			(font
@@
 	(label "A8"
 		(at 46.355 81.28 0)
-		(fields_autoplaced yes)
 		(effects
 			(font
@@
 	(label "A5"
 		(at 46.355 73.66 0)
-		(fields_autoplaced yes)
 		(effects
 			(font
@@
 	(label "A0"
 		(at 46.355 60.96 0)
-		(fields_autoplaced yes)
 		(effects
 			(font
@@
 	(label "A1"
 		(at 46.355 63.5 0)
-		(fields_autoplaced yes)
 		(effects
 			(font
@@
 	(label "D2"
 		(at 46.355 106.68 0)
-		(fields_autoplaced yes)
 		(effects
 			(font
@@
 	(label "D7"
 		(at 46.355 119.38 0)
-		(fields_autoplaced yes)
 		(effects
 			(font
@@
 	(label "D4"
 		(at 46.355 111.76 0)
-		(fields_autoplaced yes)
 		(effects
 			(font
@@
 	(label "A6"
 		(at 46.355 76.2 0)
-		(fields_autoplaced yes)
 		(effects
 			(font
@@
 	(label "WR"
 		(at 46.355 53.34 0)
-		(fields_autoplaced yes)
 		(effects
 			(font
@@
 	(label "A2"
 		(at 46.355 66.04 0)
-		(fields_autoplaced yes)
 		(effects
 			(font
@@
 	(label "A7"
 		(at 46.355 78.74 0)
-		(fields_autoplaced yes)
 		(effects
 			(font
@@
 	(label "A4"
 		(at 46.355 71.12 0)
-		(fields_autoplaced yes)
 		(effects
 			(font
@@
 	(label "VIN"
 		(at 46.355 124.46 0)
-		(fields_autoplaced yes)
 		(effects
 			(font
@@
 	(label "A15"
 		(at 46.355 99.06 0)
-		(fields_autoplaced yes)
 		(effects
 			(font
@@
 	(label "A3"
 		(at 46.355 68.58 0)
-		(fields_autoplaced yes)
 		(effects
 			(font
@@
 			)
 		)
-		(property "Value" "Crystal_Small"
+		(property "Value" "8.388608MHZ"
 			(at 127.889 102.8121 90)
 			(effects
@@
 		(unit 1)
 		(exclude_from_sim no)
-		(in_bom yes)
+		(in_bom no)
 		(on_board yes)
 		(dnp no)
@@
 		(unit 2)
 		(exclude_from_sim no)
-		(in_bom yes)
+		(in_bom no)
 		(on_board yes)
 		(dnp no)
@@
 		(in_bom yes)
 		(on_board yes)
-		(dnp no)
+		(dnp yes)
 		(property "Reference" "C46"
 			(at 252.095 37.465 0)
@@
 			)
 		)
-		(property "Value" "~"
+		(property "Value" "DNP"
 			(at 251.8791 38.6834 0)
 			(effects
@@
 		(unit 1)
 		(exclude_from_sim no)
-		(in_bom yes)
+		(in_bom no)
 		(on_board yes)
 		(dnp no)
@@
 			)
 		)
-		(property "Value" "~"
+		(property "Value" "CGB SRAM"
 			(at 174.625 59.69 0)
 			(effects
@@
 		(at 121.285 128.905)
 		(size 12.7 13.97)
+		(exclude_from_sim no)
+		(in_bom yes)
+		(on_board yes)
+		(dnp no)
 		(fields_autoplaced yes)
 		(stroke
@@
 		(at 243.205 61.595)
 		(size 12.7 74.295)
+		(exclude_from_sim no)
+		(in_bom yes)
+		(on_board yes)
+		(dnp no)
 		(fields_autoplaced yes)
 		(stroke
@@
 		(at 122.555 61.595)
 		(size 12.7 21.59)
+		(exclude_from_sim no)
+		(in_bom yes)
+		(on_board yes)
+		(dnp no)
 		(fields_autoplaced yes)
 		(stroke
@@
 		(at 121.285 151.765)
 		(size 13.335 17.78)
+		(exclude_from_sim no)
+		(in_bom yes)
+		(on_board yes)
+		(dnp no)
 		(fields_autoplaced yes)
 		(stroke
@@
 		(at 122.555 86.995)
 		(size 12.7 6.35)
+		(exclude_from_sim no)
+		(in_bom yes)
+		(on_board yes)
+		(dnp no)
 		(fields_autoplaced yes)
 		(stroke
@@
 		)
 	)
+	(embedded_fonts no)
 )
