File: KiCad Files/cgb_power.kicad_sch (KiCad schematic)
At the start: 24 parts, among them Q2 2SC4081, U5 DC-DC

Commit message: fixed some BOM stuff
Parts:
- P4, SW1, U5, U7: now left out of the parts list
Other:
- title: CGB Reverse Engineer -> Yet Another Pocket Color (YAP)
Changed lines of the file:
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@@
 (kicad_sch
-	(version 20231120)
+	(version 20250114)
 	(generator "eeschema")
-	(generator_version "8.0")
+	(generator_version "9.0")
 	(paper "A4")
 	(title_block
-		(title "CGB Reverse Engineer")
+		(title "Yet Another Pocket Color (YAP)")
 		(company "NatalieTheNerd.com")
 	)
+	(rectangle
+		(start 121.92 93.98)
+		(end 160.655 142.24)
+		(stroke
+			(width 0)
+			(type dash)
+		)
+		(fill
+			(type none)
+		)
+	)
+	(text "NOTES:"
+		(exclude_from_sim no)
+		(at 55.88 137.16 0)
+		(effects
+			(font
+				(size 3 3)
+				(thickness 0.6)
+				(bold yes)
+			)
+			(justify left bottom)
+		)
+	)
+	(text "D2 80V 1.2V@100mA"
+		(exclude_from_sim no)
+		(at 57.15 154.94 0)
+		(effects
+			(font
+				(size 1.27 1.27)
+			)
+			(justify left bottom)
+			(href "https://github.com/nataliethenerd/CGB_ReverseEngineer/blob/main/datasheets/1SS355.pdf")
+		)
+	)
+	(text "EM6-8 220Ω@100MHz ferrite bead"
+		(exclude_from_sim no)
+		(at 57.15 149.86 0)
+		(effects
+			(font
+				(size 1.27 1.27)
+			)
+			(justify left bottom)
+		)
+	)
+	(text "EM10 Common mode filter "
+		(exclude_from_sim no)
+		(at 57.15 144.78 0)
+		(effects
+			(font
+				(size 1.27 1.27)
+			)
+			(justify left bottom)
+			(href "https://github.com/nataliethenerd/CGB_ReverseEngineer/blob/main/datasheets/ACM4532-801-2P.pdf")
+		)
+	)
+	(text "F1,2 fuse 1A 50V "
+		(exclude_from_sim no)
+		(at 57.15 147.32 0)
+		(effects
+			(font
+				(size 1.27 1.27)
+			)
+			(justify left bottom)
+		)
+	)
+	(text "Power LED\n"
+		(exclude_from_sim no)
+		(at 128.27 97.79 0)
+		(effects
+			(font
+				(size 1.27 1.27)
+				(italic yes)
+			)
+			(justify left bottom)
+		)
+	)
+	(text "Q2 NPN transistor"
+		(exclude_from_sim no)
+		(at 57.15 152.4 0)
+		(effects
+			(font
+				(size 1.27 1.27)
+			)
+			(justify left bottom)
+			(href "https://github.com/nataliethenerd/CGB_ReverseEngineer/blob/main/datasheets/2SC4081.pdf")
+		)
+	)
+	(text "VCC = battery voltage"
+		(exclude_from_sim no)
+		(at 55.88 142.24 0)
+		(effects
+			(font
+				(size 2 2)
+				(italic yes)
+			)
+			(justify left bottom)
+		)
+	)
 	(junction
 		(at 140.97 87.63)
@@
 		)
 	)
-	(rectangle
-		(start 121.92 93.98)
-		(end 160.655 142.24)
-		(stroke
-			(width 0)
-			(type dash)
-		)
-		(fill
-			(type none)
-		)
-	)
-	(text "NOTES:"
-		(exclude_from_sim no)
-		(at 55.88 137.16 0)
-		(effects
-			(font
-				(size 3 3)
-				(thickness 0.6)
-				(bold yes)
-			)
-			(justify left bottom)
-		)
-	)
-	(text "D2 80V 1.2V@100mA"
-		(exclude_from_sim no)
-		(at 57.15 154.94 0)
-		(effects
-			(font
-				(size 1.27 1.27)
-			)
-			(justify left bottom)
-			(href "https://github.com/nataliethenerd/CGB_ReverseEngineer/blob/main/datasheets/1SS355.pdf")
-		)
-	)
-	(text "EM6-8 220Ω@100MHz ferrite bead"
-		(exclude_from_sim no)
-		(at 57.15 149.86 0)
-		(effects
-			(font
-				(size 1.27 1.27)
-			)
-			(justify left bottom)
-		)
-	)
-	(text "EM10 Common mode filter "
-		(exclude_from_sim no)
-		(at 57.15 144.78 0)
-		(effects
-			(font
-				(size 1.27 1.27)
-			)
-			(justify left bottom)
-			(href "https://github.com/nataliethenerd/CGB_ReverseEngineer/blob/main/datasheets/ACM4532-801-2P.pdf")
-		)
-	)
-	(text "F1,2 fuse 1A 50V "
-		(exclude_from_sim no)
-		(at 57.15 147.32 0)
-		(effects
-			(font
-				(size 1.27 1.27)
-			)
-			(justify left bottom)
-		)
-	)
-	(text "Power LED\n"
-		(exclude_from_sim no)
-		(at 128.27 97.79 0)
-		(effects
-			(font
-				(size 1.27 1.27)
-				(italic yes)
-			)
-			(justify left bottom)
-		)
-	)
-	(text "Q2 NPN transistor"
-		(exclude_from_sim no)
-		(at 57.15 152.4 0)
-		(effects
-			(font
-				(size 1.27 1.27)
-			)
-			(justify left bottom)
-			(href "https://github.com/nataliethenerd/CGB_ReverseEngineer/blob/main/datasheets/2SC4081.pdf")
-		)
-	)
-	(text "VCC = battery voltage"
-		(exclude_from_sim no)
-		(at 55.88 142.24 0)
-		(effects
-			(font
-				(size 2 2)
-				(italic yes)
-			)
-			(justify left bottom)
-		)
-	)
 	(symbol
 		(lib_id "Device:D_Small")
@@
 		(unit 1)
 		(exclude_from_sim no)
-		(in_bom yes)
+		(in_bom no)
 		(on_board yes)
 		(dnp no)
@@
 		(unit 1)
 		(exclude_from_sim no)
-		(in_bom yes)
+		(in_bom no)
 		(on_board yes)
 		(dnp no)
@@
 		(unit 1)
 		(exclude_from_sim no)
-		(in_bom yes)
+		(in_bom no)
 		(on_board yes)
 		(dnp no)
@@
 		(unit 1)
 		(exclude_from_sim no)
-		(in_bom yes)
+		(in_bom no)
 		(on_board yes)
 		(dnp no)
