File: KiCad Files/cgb_screen.kicad_sch (KiCad schematic)
At the start: 7 parts, among them J1 Conn_01x04

Commit message: fixed some BOM stuff
Parts:
- J1: value Conn_01x04 -> Thumbwheel Toggle Switch
- P2: value ~ -> FPC 50 Pin 0.5 Pitch (top contacts)
- TST3: now left out of the parts list
Other:
- note removed: "Original screen circuitry"
- title: CGB Reverse Engineer -> Yet Another Pocket Color (YAP)
